File: usb-switch/upstream_port.kicad_sch (KiCad schematic)
At the start: 19 parts, among them J1 USB_C_Receptacle, U5 FUSB307BMPX, U6 HD3SS3212IRKSR, U7 TUSB8043AIRGCR

Commit message: Starting to look closer to completion
Parts:
- J1: TYPE (none) -> UPSTREAM
- renumbered U7 to U10, U5 to U8, U6 to U9
Other:
- title: (none) -> Upstream Port Module
Changed lines of the file:
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@@
 (kicad_sch (version 20230121) (generator eeschema)
   (paper "A4")
+  (title_block
+    (title "Upstream Port Module")
+  )
   (bus_alias "CCBUS" (members "CC1" "CC2"))
   (bus_alias "I2C" (members "SCL" "SDA"))
@@
     (effects (font (size 1.27 1.27)) (justify right bottom))
   )
-  (label "I2C_A.SCL" (at 259.08 104.14 90)
+  (label "I2C_A.SCL" (at 259.08 104.14 90) (fields_autoplaced)
     (effects (font (size 1.27 1.27)) (justify left bottom))
   )
@@
     (effects (font (size 1.27 1.27)) (justify left bottom))
   )
-  (label "I2C_A.SDA" (at 262.89 104.14 90)
+  (label "I2C_A.SDA" (at 262.89 104.14 90) (fields_autoplaced)
     (effects (font (size 1.27 1.27)) (justify left bottom))
   )
@@
   (symbol (lib_id "Interface_USB:FUSB307BMPX") (at 73.66 34.29 180) (unit 1)
     (in_bom yes) (on_board yes) (dnp no) (fields_autoplaced)
-    (property "Reference" "U5" (at 74.0059 16.51 0)
+    (property "Reference" "U8" (at 74.0059 16.51 0)
       (effects (font (size 1.27 1.27)) (justify right))
     )
@@
       (project "usb-switch"
         (path "/e9ad9249-a54d-4a1a-ae9a-437037ccf4af/c506baa8-3fb8-4c1e-b12b-db5db1a9e333"
-          (reference "U5") (unit 1)
-        )
-        (path "/e9ad9249-a54d-4a1a-ae9a-437037ccf4af/3ea6c733-b856-496c-b2e5-3fc306de3a0b"
           (reference "U8") (unit 1)
         )
-        (path "/e9ad9249-a54d-4a1a-ae9a-437037ccf4af/30337322-f4e8-4295-b2ae-df4bab4dbabb"
+        (path "/e9ad9249-a54d-4a1a-ae9a-437037ccf4af/3ea6c733-b856-496c-b2e5-3fc306de3a0b"
           (reference "U11") (unit 1)
         )
-        (path "/e9ad9249-a54d-4a1a-ae9a-437037ccf4af/96db75ba-e971-4b24-b1c6-9f76512c9163"
+        (path "/e9ad9249-a54d-4a1a-ae9a-437037ccf4af/30337322-f4e8-4295-b2ae-df4bab4dbabb"
           (reference "U14") (unit 1)
+        )
+        (path "/e9ad9249-a54d-4a1a-ae9a-437037ccf4af/96db75ba-e971-4b24-b1c6-9f76512c9163"
+          (reference "U17") (unit 1)
         )
       )
@@
   (symbol (lib_id "project-library:HD3SS3212IRKSR") (at 88.9 101.6 180) (unit 1)
     (in_bom yes) (on_board yes) (dnp no) (fields_autoplaced)
-    (property "Reference" "U6" (at 88.9 68.58 0)
+    (property "Reference" "U9" (at 88.9 68.58 0)
       (effects (font (size 1.524 1.524)))
     )
@@
       (project "usb-switch"
         (path "/e9ad9249-a54d-4a1a-ae9a-437037ccf4af/c506baa8-3fb8-4c1e-b12b-db5db1a9e333"
-          (reference "U6") (unit 1)
-        )
-        (path "/e9ad9249-a54d-4a1a-ae9a-437037ccf4af/3ea6c733-b856-496c-b2e5-3fc306de3a0b"
           (reference "U9") (unit 1)
         )
-        (path "/e9ad9249-a54d-4a1a-ae9a-437037ccf4af/30337322-f4e8-4295-b2ae-df4bab4dbabb"
+        (path "/e9ad9249-a54d-4a1a-ae9a-437037ccf4af/3ea6c733-b856-496c-b2e5-3fc306de3a0b"
           (reference "U12") (unit 1)
         )
-        (path "/e9ad9249-a54d-4a1a-ae9a-437037ccf4af/96db75ba-e971-4b24-b1c6-9f76512c9163"
+        (path "/e9ad9249-a54d-4a1a-ae9a-437037ccf4af/30337322-f4e8-4295-b2ae-df4bab4dbabb"
           (reference "U15") (unit 1)
+        )
+        (path "/e9ad9249-a54d-4a1a-ae9a-437037ccf4af/96db75ba-e971-4b24-b1c6-9f76512c9163"
+          (reference "U18") (unit 1)
         )
       )
@@
   (symbol (lib_id "project-library:TUSB8043AIRGCR") (at 127 36.83 0) (unit 1)
     (in_bom yes) (on_board yes) (dnp no) (fields_autoplaced)
-    (property "Reference" "U7" (at 190.5 26.67 0)
+    (property "Reference" "U10" (at 190.5 26.67 0)
       (effects (font (size 1.524 1.524)))
     )
@@
       (project "usb-switch"
         (path "/e9ad9249-a54d-4a1a-ae9a-437037ccf4af/c506baa8-3fb8-4c1e-b12b-db5db1a9e333"
-          (reference "U7") (unit 1)
-        )
-        (path "/e9ad9249-a54d-4a1a-ae9a-437037ccf4af/3ea6c733-b856-496c-b2e5-3fc306de3a0b"
           (reference "U10") (unit 1)
         )
-        (path "/e9ad9249-a54d-4a1a-ae9a-437037ccf4af/30337322-f4e8-4295-b2ae-df4bab4dbabb"
+        (path "/e9ad9249-a54d-4a1a-ae9a-437037ccf4af/3ea6c733-b856-496c-b2e5-3fc306de3a0b"
           (reference "U13") (unit 1)
         )
-        (path "/e9ad9249-a54d-4a1a-ae9a-437037ccf4af/96db75ba-e971-4b24-b1c6-9f76512c9163"
+        (path "/e9ad9249-a54d-4a1a-ae9a-437037ccf4af/30337322-f4e8-4295-b2ae-df4bab4dbabb"
           (reference "U16") (unit 1)
+        )
+        (path "/e9ad9249-a54d-4a1a-ae9a-437037ccf4af/96db75ba-e971-4b24-b1c6-9f76512c9163"
+          (reference "U19") (unit 1)
         )
       )
@@
     )
     (property "Datasheet" "https://www.usb.org/sites/default/files/documents/usb_type-c.zip" (at 27.94 95.25 0)
+      (effects (font (size 1.27 1.27)) hide)
+    )
+    (property "TYPE" "UPSTREAM" (at 24.13 95.25 0)
       (effects (font (size 1.27 1.27)) hide)
     )
@@
   (symbol (lib_name "TUSB8043AIRGCR_1") (lib_id "project-library:TUSB8043AIRGCR") (at 116.84 148.59 0) (unit 2)
     (in_bom yes) (on_board yes) (dnp no)
-    (property "Reference" "U7" (at 198.12 137.16 0)
+    (property "Reference" "U10" (at 198.12 137.16 0)
       (effects (font (size 1.524 1.524)) hide)
     )
@@
       (project "usb-switch"
         (path "/e9ad9249-a54d-4a1a-ae9a-437037ccf4af/c506baa8-3fb8-4c1e-b12b-db5db1a9e333"
-          (reference "U7") (unit 2)
-        )
-        (path "/e9ad9249-a54d-4a1a-ae9a-437037ccf4af/3ea6c733-b856-496c-b2e5-3fc306de3a0b"
           (reference "U10") (unit 2)
         )
-        (path "/e9ad9249-a54d-4a1a-ae9a-437037ccf4af/30337322-f4e8-4295-b2ae-df4bab4dbabb"
+        (path "/e9ad9249-a54d-4a1a-ae9a-437037ccf4af/3ea6c733-b856-496c-b2e5-3fc306de3a0b"
           (reference "U13") (unit 2)
         )
-        (path "/e9ad9249-a54d-4a1a-ae9a-437037ccf4af/96db75ba-e971-4b24-b1c6-9f76512c9163"
+        (path "/e9ad9249-a54d-4a1a-ae9a-437037ccf4af/30337322-f4e8-4295-b2ae-df4bab4dbabb"
           (reference "U16") (unit 2)
         )
-      )
+        (path "/e9ad9249-a54d-4a1a-ae9a-437037ccf4af/96db75ba-e971-4b24-b1c6-9f76512c9163"
+          (reference "U19") (unit 2)
+        )
+      )
