File: usb-switch/usb-switch.kicad_pcb (KiCad board)
At the start: 2 copper layers, 0 parts

Commit message: Starting to look closer to completion
Parts:
- added C1: 0.1uF, Capacitor_SMD:C_0201_0603Metric, F.Cu at (88.6, 130.9)
- added C10: 0.1uF, Capacitor_SMD:C_0201_0603Metric, F.Cu at (91.1, 136.2)
- added C11: 0.1uF, Capacitor_SMD:C_0201_0603Metric, F.Cu at (91.1, 137.9)
- added C12: 0.1uF, Capacitor_SMD:C_0201_0603Metric, F.Cu at (91.1, 139.7)
- added C13: 0.1uF, Capacitor_SMD:C_0201_0603Metric, F.Cu at (124.2, 117.5)
- added C14: 0.1uF, Capacitor_SMD:C_0201_0603Metric, F.Cu at (124.2, 119.2)
- added C15: 0.1uF, Capacitor_SMD:C_0201_0603Metric, F.Cu at (124.2, 121.0)
- added C16: 0.1uF, Capacitor_SMD:C_0201_0603Metric, F.Cu at (124.2, 122.7)
- added C17: 0.1uF, Capacitor_SMD:C_0201_0603Metric, F.Cu at (124.2, 124.5)
- added C18: 0.1uF, Capacitor_SMD:C_0201_0603Metric, F.Cu at (124.2, 126.2)
- added C19: 0.1uF, Capacitor_SMD:C_0201_0603Metric, F.Cu at (126.7, 117.5)
- added C2: 0.1uF, Capacitor_SMD:C_0201_0603Metric, F.Cu at (88.6, 132.7)
- added C20: 0.1uF, Capacitor_SMD:C_0201_0603Metric, F.Cu at (126.7, 119.2)
- added C21: 0.1uF, Capacitor_SMD:C_0201_0603Metric, F.Cu at (126.7, 121.0)
- added C22: 0.1uF, Capacitor_SMD:C_0201_0603Metric, F.Cu at (126.7, 122.7)
- added C23: 0.1uF, Capacitor_SMD:C_0201_0603Metric, F.Cu at (126.7, 124.5)
- added C24: 0.1uF, Capacitor_SMD:C_0201_0603Metric, F.Cu at (126.7, 126.2)
- added C25: 0.1uF, Capacitor_SMD:C_0201_0603Metric, F.Cu at (149.6, 118.2)
- added C26: 0.1uF, Capacitor_SMD:C_0201_0603Metric, F.Cu at (149.6, 120.0)
- added C27: 0.1uF, Capacitor_SMD:C_0201_0603Metric, F.Cu at (149.6, 121.8)
- added C28: 0.1uF, Capacitor_SMD:C_0201_0603Metric, F.Cu at (149.6, 123.5)
- added C29: 0.1uF, Capacitor_SMD:C_0201_0603Metric, F.Cu at (149.6, 125.2)
- added C3: 0.1uF, Capacitor_SMD:C_0201_0603Metric, F.Cu at (88.6, 134.4)
- added C30: 0.1uF, Capacitor_SMD:C_0201_0603Metric, F.Cu at (149.6, 127.0)
- added C31: 0.1uF, Capacitor_SMD:C_0201_0603Metric, F.Cu at (152.1, 118.2)
- added C32: 0.1uF, Capacitor_SMD:C_0201_0603Metric, F.Cu at (152.1, 120.0)
- added C33: 0.1uF, Capacitor_SMD:C_0201_0603Metric, F.Cu at (152.1, 121.8)
- added C34: 0.1uF, Capacitor_SMD:C_0201_0603Metric, F.Cu at (152.1, 123.5)
- added C35: 0.1uF, Capacitor_SMD:C_0201_0603Metric, F.Cu at (152.1, 125.2)
- added C36: 0.1uF, Capacitor_SMD:C_0201_0603Metric, F.Cu at (152.1, 127.0)
- added C37: 0.1uF, Capacitor_SMD:C_0201_0603Metric, F.Cu at (164.8, 118.2)
- added C38: 0.1uF, Capacitor_SMD:C_0201_0603Metric, F.Cu at (164.8, 120.0)
- added C39: 0.1uF, Capacitor_SMD:C_0201_0603Metric, F.Cu at (164.8, 121.8)
- added C4: 0.1uF, Capacitor_SMD:C_0201_0603Metric, F.Cu at (88.6, 136.2)
- added C40: 0.1uF, Capacitor_SMD:C_0201_0603Metric, F.Cu at (164.8, 123.5)
- added C41: 0.1uF, Capacitor_SMD:C_0201_0603Metric, F.Cu at (164.8, 125.2)
- added C42: 0.1uF, Capacitor_SMD:C_0201_0603Metric, F.Cu at (164.8, 127.0)
- added C43: 0.1uF, Capacitor_SMD:C_0201_0603Metric, F.Cu at (167.3, 118.2)
- added C44: 0.1uF, Capacitor_SMD:C_0201_0603Metric, F.Cu at (167.3, 120.0)
- added C45: 0.1uF, Capacitor_SMD:C_0201_0603Metric, F.Cu at (167.3, 121.8)
- added C46: 0.1uF, Capacitor_SMD:C_0201_0603Metric, F.Cu at (167.3, 123.5)
- added C47: 0.1uF, Capacitor_SMD:C_0201_0603Metric, F.Cu at (167.3, 125.2)
- added C48: 0.1uF, Capacitor_SMD:C_0201_0603Metric, F.Cu at (167.3, 127.0)
- added C49: 0.1uF, Capacitor_SMD:C_0402_1005Metric, F.Cu at (136.8, 67.3)
- added C5: 0.1uF, Capacitor_SMD:C_0201_0603Metric, F.Cu at (88.6, 137.9)
- added C50: 0.1uF, Capacitor_SMD:C_0402_1005Metric, F.Cu at (136.8, 69.3)
- added C51: 0.1uF, Capacitor_SMD:C_0402_1005Metric, F.Cu at (116.4, 71.7)
- added C52: 0.1uF, Capacitor_SMD:C_0402_1005Metric, F.Cu at (116.4, 73.7)
- added C53: 0.1uF, Capacitor_SMD:C_0402_1005Metric, F.Cu at (162.3, 67.3)
- added C54: 0.1uF, Capacitor_SMD:C_0402_1005Metric, F.Cu at (162.3, 69.3)
- added C55: 0.1uF, Capacitor_SMD:C_0402_1005Metric, F.Cu at (111.3, 67.3)
- added C56: 0.1uF, Capacitor_SMD:C_0402_1005Metric, F.Cu at (111.3, 69.3)
- added C6: 0.1uF, Capacitor_SMD:C_0201_0603Metric, F.Cu at (88.6, 139.7)
- added C7: 0.1uF, Capacitor_SMD:C_0201_0603Metric, F.Cu at (91.1, 130.9)
- added C8: 0.1uF, Capacitor_SMD:C_0201_0603Metric, F.Cu at (91.1, 132.7)
- added C9: 0.1uF, Capacitor_SMD:C_0201_0603Metric, F.Cu at (91.1, 134.4)
- added J1: USB_C_Receptacle, Connector_USB:USB_C_Receptacle_Amphenol_12401548E4-2A, F.Cu at (101.5, 157.5)
- added J2: USB_C_Receptacle, Connector_USB:USB_C_Receptacle_Amphenol_12401548E4-2A, F.Cu at (124.5, 157.2)
- added J3: USB_C_Receptacle, Connector_USB:USB_C_Receptacle_Amphenol_12401548E4-2A, F.Cu at (147.3, 157.2)
- added J4: USB_C_Receptacle, Connector_USB:USB_C_Receptacle_Amphenol_12401548E4-2A, F.Cu at (169.2, 157.7)
- added J5: USB_C_Receptacle, Connector_USB:USB_C_Receptacle_Amphenol_12401548E4-2A, F.Cu at (139.7, 27.9)
- added J6: USB_C_Receptacle, Connector_USB:USB_C_Receptacle_Amphenol_12401548E4-2A, F.Cu at (89.5, 28.2)
- added J7: USB_C_Receptacle, Connector_USB:USB_C_Receptacle_Amphenol_12401548E4-2A, F.Cu at (165.1, 27.9)
- added J8: USB_C_Receptacle, Connector_USB:USB_C_Receptacle_Amphenol_12401548E4-2A, F.Cu at (114.3, 27.9)
- added R1: 12k, Resistor_SMD:R_0201_0603Metric, F.Cu at (93.5, 130.9)
- added R10: 12k, Resistor_SMD:R_0201_0603Metric, F.Cu at (169.7, 118.2)
- added R11: 9.53k, Resistor_SMD:R_0201_0603Metric, F.Cu at (169.7, 120.0)
- added R12: 10k, Resistor_SMD:R_0201_0603Metric, F.Cu at (169.7, 121.8)
- added R13: 10k, Resistor_SMD:R_0201_0603Metric, F.Cu at (147.1, 61.1)
- added R14: 10k, Resistor_SMD:R_0201_0603Metric, F.Cu at (147.1, 62.9)
- added R15: 10k, Resistor_SMD:R_0201_0603Metric, F.Cu at (147.1, 64.6)
- added R16: 10k, Resistor_SMD:R_0201_0603Metric, F.Cu at (147.1, 66.4)
- added R17: 10k, Resistor_SMD:R_0201_0603Metric, F.Cu at (101.8, 58.1)
- added R18: 10k, Resistor_SMD:R_0201_0603Metric, F.Cu at (100.0, 58.1)
- added R19: 10k, Resistor_SMD:R_0201_0603Metric, F.Cu at (98.3, 58.1)
- added R2: 9.53k, Resistor_SMD:R_0201_0603Metric, F.Cu at (93.5, 132.7)
- added R20: 10k, Resistor_SMD:R_0201_0603Metric, F.Cu at (96.5, 58.1)
- added R21: 10k, Resistor_SMD:R_0201_0603Metric, F.Cu at (172.6, 61.1)
- added R22: 10k, Resistor_SMD:R_0201_0603Metric, F.Cu at (172.6, 62.9)
- added R23: 10k, Resistor_SMD:R_0201_0603Metric, F.Cu at (172.6, 64.6)
- added R24: 10k, Resistor_SMD:R_0201_0603Metric, F.Cu at (172.6, 66.4)
- added R25: 10k, Resistor_SMD:R_0201_0603Metric, F.Cu at (121.6, 61.1)
- added R26: 10k, Resistor_SMD:R_0201_0603Metric, F.Cu at (121.6, 62.9)
- added R27: 10k, Resistor_SMD:R_0201_0603Metric, F.Cu at (121.6, 64.6)
- added R28: 10k, Resistor_SMD:R_0201_0603Metric, F.Cu at (121.6, 66.4)
- added R3: 10k, Resistor_SMD:R_0201_0603Metric, F.Cu at (93.5, 134.4)
- added R4: 12k, Resistor_SMD:R_0201_0603Metric, F.Cu at (129.1, 117.5)
- added R5: 9.53k, Resistor_SMD:R_0201_0603Metric, F.Cu at (129.1, 119.2)
- added R6: 10k, Resistor_SMD:R_0201_0603Metric, F.Cu at (129.1, 121.0)
- added R7: 12k, Resistor_SMD:R_0201_0603Metric, F.Cu at (154.5, 118.2)
- added R8: 9.53k, Resistor_SMD:R_0201_0603Metric, F.Cu at (154.5, 120.0)
- added R9: 10k, Resistor_SMD:R_0201_0603Metric, F.Cu at (154.5, 121.8)
- added U1: LTC4317, Package_DFN_QFN:DFN-16-1EP_3x5mm_P0.5mm_EP1.66x4.4mm, F.Cu at (101.8, 102.9)
- added U10: TUSB8043AIRGCR, Library:VQFN64_RGC_TEX, F.Cu at (102.8, 135.3)
- added U11: FUSB307BMPX, Package_DFN_QFN:WQFN-16-1EP_3x3mm_P0.5mm_EP1.75x1.75mm, F.Cu at (134.9, 153.5)
- added U12: HD3SS3212IRKSR, Library:RKS0020A, F.Cu at (125.3, 145.9)
- added U13: TUSB8043AIRGCR, Library:VQFN64_RGC_TEX, F.Cu at (125.8, 135.3)
- added U14: FUSB307BMPX, Package_DFN_QFN:WQFN-16-1EP_3x3mm_P0.5mm_EP1.75x1.75mm, F.Cu at (156.7, 153.5)
- added U15: HD3SS3212IRKSR, Library:RKS0020A, F.Cu at (148.1, 145.9)
- added U16: TUSB8043AIRGCR, Library:VQFN64_RGC_TEX, F.Cu at (145.4, 135.9)
- added U17: FUSB307BMPX, Package_DFN_QFN:WQFN-16-1EP_3x3mm_P0.5mm_EP1.75x1.75mm, F.Cu at (179.6, 156.0)
- added U18: HD3SS3212IRKSR, Library:RKS0020A, F.Cu at (168.0, 147.6)
- added U19: TUSB8043AIRGCR, Library:VQFN64_RGC_TEX, F.Cu at (165.7, 135.9)
- added U2: LTC4317, Package_DFN_QFN:DFN-16-1EP_3x5mm_P0.5mm_EP1.66x4.4mm, F.Cu at (106.9, 102.9)
- added U20: max4999etj+, Library:21-0140_T3255+4_MXM, F.Cu at (150.0, 44.0)
- added U21: HD3SS3412RUAR, Library:RUA0042A, F.Cu at (133.8, 41.7)
- added U22: TCA9534, Package_SO:SOIC-16_4.55x10.3mm_P1.27mm, F.Cu at (141.5, 53.5)
- added U23: HD3SS3212IRKSR, Library:RKS0020A, F.Cu at (140.5, 42.0)
- added U24: HD3SS3212IRKSR, Library:RKS0020A, F.Cu at (139.3, 37.8)
- added U25: FUSB307BMPX, Package_DFN_QFN:WQFN-16-1EP_3x3mm_P0.5mm_EP1.75x1.75mm, F.Cu at (132.7, 69.0)
- added U26: max4999etj+, Library:21-0140_T3255+4_MXM, F.Cu at (81.4, 59.7)
- added U27: HD3SS3412RUAR, Library:RUA0042A, F.Cu at (90.4, 50.0)
- added U28: TCA9534, Package_SO:SOIC-16_4.55x10.3mm_P1.27mm, F.Cu at (95.9, 66.8)
- added U29: HD3SS3212IRKSR, Library:RKS0020A, F.Cu at (89.3, 42.9)
- added U3: PCA9537, Package_SO:TSSOP-10_3x3mm_P0.5mm, F.Cu at (102.8, 108.6)
- added U30: HD3SS3212IRKSR, Library:RKS0020A, F.Cu at (89.3, 37.8)
- added U31: FUSB307BMPX, Package_DFN_QFN:WQFN-16-1EP_3x3mm_P0.5mm_EP1.75x1.75mm, F.Cu at (79.5, 37.0)
- added U32: max4999etj+, Library:21-0140_T3255+4_MXM, F.Cu at (177.9, 44.0)
- added U33: HD3SS3412RUAR, Library:RUA0042A, F.Cu at (158.3, 44.6)
- added U34: TCA9534, Package_SO:SOIC-16_4.55x10.3mm_P1.27mm, F.Cu at (167.0, 53.5)
- added U35: HD3SS3212IRKSR, Library:RKS0020A, F.Cu at (165.9, 42.0)
- added U36: HD3SS3212IRKSR, Library:RKS0020A, F.Cu at (165.5, 37.8)
- added U37: FUSB307BMPX, Package_DFN_QFN:WQFN-16-1EP_3x3mm_P0.5mm_EP1.75x1.75mm, F.Cu at (158.2, 69.0)
- added U38: max4999etj+, Library:21-0140_T3255+4_MXM, F.Cu at (106.8, 49.1)
- added U39: HD3SS3412RUAR, Library:RUA0042A, F.Cu at (120.8, 42.4)
- added U4: RP2040, Package_DFN_QFN:QFN-56-1EP_7x7mm_P0.4mm_EP3.2x3.2mm, F.Cu at (86.3, 98.2)
- added U40: TCA9534, Package_SO:SOIC-16_4.55x10.3mm_P1.27mm, F.Cu at (116.0, 53.5)
- added U41: HD3SS3212IRKSR, Library:RKS0020A, F.Cu at (107.2, 41.0)
- added U42: HD3SS3212IRKSR, Library:RKS0020A, F.Cu at (115.1, 36.7)
- added U43: FUSB307BMPX, Package_DFN_QFN:WQFN-16-1EP_3x3mm_P0.5mm_EP1.75x1.75mm, F.Cu at (104.9, 34.1)
- added U5: LTC4317, Package_DFN_QFN:DFN-16-1EP_3x5mm_P0.5mm_EP1.66x4.4mm, F.Cu at (111.9, 102.9)
- added U6: PCA9537, Package_SO:TSSOP-10_3x3mm_P0.5mm, F.Cu at (102.8, 113.2)
- added U7: LTC4317, Package_DFN_QFN:DFN-16-1EP_3x5mm_P0.5mm_EP1.66x4.4mm, F.Cu at (117.0, 102.9)
- added U8: FUSB307BMPX, Package_DFN_QFN:WQFN-16-1EP_3x3mm_P0.5mm_EP1.75x1.75mm, F.Cu at (110.3, 154.2)
- added U9: HD3SS3212IRKSR, Library:RKS0020A, F.Cu at (102.3, 146.2)
- added X1: ASDMB-24MHz, Oscillator:Oscillator_SMD_Abracon_ASDMB-4Pin_2.5x2.0mm, F.Cu at (108.3, 117.5)
Other:
- board outline added: 114.3 x 134.6 mm
