File: usb-switch/downstream_port.kicad_sch (KiCad schematic)
At the start: 10 parts, among them J5 USB_C_Receptacle, U17 max4999etj+, U18 HD3SS3412RUAR, U19 HD3SS3212IRKSR, U20 HD3SS3212IRKSR, U21 FUSB307BMPX, U22 TCA9534

Commit message: Starting to look closer to completion
Parts:
- added R14, R15, R17: 10k, Resistor_SMD:R_0201_0603Metric, symbol Device:R_Small
- J5: TYPE (none) -> DOWNSTREAM
- R16: renamed from R13; footprint (none) -> Resistor_SMD:R_0201_0603Metric
- U20: renamed from U17; footprint 21-0140_T3255+4_MXM -> Library:21-0140_T3255+4_MXM
- U21: renamed from U18; footprint RUA0042A -> Library:RUA0042A
- U22: footprint (none) -> Package_SO:SOIC-16_4.55x10.3mm_P1.27mm
- renumbered U19 to U23, U20 to U24, U21 to U25
Connections:
- net DFP_VBUS: now also U25.2 (VCONN); no longer U25.6 (VBUS)
- net GND: now also U22.8 (GND), R14.1, R15.1, R17.1
- net at U22.1 (A0): now also R17.2
- net CONTROL.INT: now reaches U22.13 (~{INT})
- net at U22.2 (A1): now also R14.2
- net at U22.3 (A2): now also R15.2
- net SCL renamed CONTROL.SCL
- net SDA renamed CONTROL.SDA
- no-connect marks 23 -> 26
Other:
- title: (none) -> Downstream Port Module
